File: PCB/Custom-Fan.kicad_pcb (KiCad board)
At the start: 2 copper layers, 52.5 x 38.5 mm, 4 parts, among them Q1 BC517, U1 XIAO-RP2040-DIP

Commit message: Add files via upload
Parts:
- removed D1: NeoPixel_THT, Crystal:Crystal_SMD_3225-4Pin_3.2x2.5mm_HandSoldering
Routing:
- net +5V: track 33.8 -> 39.4 mm, vias 0 -> 1
- net Net-(D1-DIN): track 14.1 -> 15.8 mm, vias 0 -> 1
- net GND: track 82.6 -> 81.2 mm, vias 2 -> 3
- net (no net): vias 0 -> 1
Other:
- board text added: "+5V"
- board text added: "DIN"
- board text added: "DON"
- board text added: "GND"
- board text added: "RGB LED"
